Commit message: pushingn the update

File: urdfs/vnymous.urdf (robot description, URDF)
Before this commit: robot vnymous, 12 links, 11 joints
Links:
- link base_link: geometry collision mesh filename=file:///home/abhiyaan-nuc/ar_ws/src/ar_sim/meshes/igvc/igvc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 scale=0.001 0.001 0.001; visual mesh filename=file:///home/abhiyaan-nuc/ar_ws/src/ar_sim/meshes/igvc/igvc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 scale=0.001 0.001 0.001
- link wheel1: geometry collision cylinder length=0.04 radius=0.12; visual mesh filename=file:///home/abhiyaan-nuc/ar_ws/src/ar_sim/meshes/igvc/igvc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 scale=0.001 0.001 0.001
- link wheel2: geometry collision cylinder length=0.04 radius=0.12; visual mesh filename=file:///home/abhiyaan-nuc/ar_ws/src/ar_sim/meshes/igvc/igvc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 scale=0.001 0.001 0.001
- link zed_camera: geometry collision mesh filename=file:///home/abhiyaan-nuc/ar_ws/src/ar_sim/meshes/igvc/zed2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; visual mesh filename=file:///home/abhiyaan-nuc/ar_ws/src/ar_sim/meshes/igvc/zed2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 scale=1 1 1
